File: example/charging_station/Mainboard_V1/Mainboard_V1.kicad_pcb (KiCad board)
At the start: 2 copper layers, 0 parts

Commit message: Update PCB
Parts:
- added C101: 100uF, Capacitor_THT:CP_Radial_D4.0mm_P1.50mm, F.Cu at (173.2, 59.5)
- added C201: 100uF, Capacitor_THT:CP_Radial_D4.0mm_P1.50mm, F.Cu at (103.0, 125.5)
- added C202: 100uF, Capacitor_THT:CP_Radial_D4.0mm_P1.50mm, F.Cu at (197.5, 108.5)
- added J102: ~, Mainboard:PogoPin, F.Cu at (131.0, 87.0)
- added J103: ~, Mainboard:PogoPin, F.Cu at (173.0, 87.0)
- added J104: Conn_01x04_Pin, Connector_PinHeader_2.54mm:PinHeader_1x04_P2.54mm_Vertical, F.Cu at (123.6, 51.5)
- added J107: Conn_01x08_Pin, Connector_PinHeader_2.54mm:PinHeader_1x08_P2.54mm_Vertical, F.Cu at (172.8, 53.0)
- added Mr201: Stepper_Motor_unipolar_6pin, Connector_PinHeader_2.54mm:PinHeader_1x06_P2.54mm_Vertical, F.Cu at (103.0, 107.3)
- added Mr202: Stepper_Motor_unipolar_6pin, Connector_PinHeader_2.54mm:PinHeader_1x06_P2.54mm_Vertical, F.Cu at (197.5, 126.7)
- added R101: 1k, Resistor_THT:R_Axial_DIN0207_L6.3mm_D2.5mm_P10.16mm_Horizontal, F.Cu at (138.6, 98.5)
- added R102: 1k, Resistor_THT:R_Axial_DIN0207_L6.3mm_D2.5mm_P10.16mm_Horizontal, F.Cu at (138.7, 94.5)
- added R103: 1k, Resistor_THT:R_Axial_DIN0207_L6.3mm_D2.5mm_P10.16mm_Horizontal, F.Cu at (161.8, 121.5)
- added R104: 1k, Resistor_THT:R_Axial_DIN0207_L6.3mm_D2.5mm_P10.16mm_Horizontal, F.Cu at (161.8, 125.5)
- added R105: 1k, Resistor_THT:R_Axial_DIN0207_L6.3mm_D2.5mm_P10.16mm_Horizontal, F.Cu at (161.9, 117.5)
- added R106: 1k, Resistor_THT:R_Axial_DIN0207_L6.3mm_D2.5mm_P10.16mm_Horizontal, F.Cu at (138.6, 102.5)
- added R107: 1k, Resistor_THT:R_Axial_DIN0207_L6.3mm_D2.5mm_P10.16mm_Horizontal, F.Cu at (125.5, 68.6)
- added R108: 1k, Resistor_THT:R_Axial_DIN0207_L6.3mm_D2.5mm_P10.16mm_Horizontal, F.Cu at (121.0, 68.6)
- added R116: 1k, Resistor_THT:R_Axial_DIN0207_L6.3mm_D2.5mm_P10.16mm_Horizontal, F.Cu at (187.0, 67.6)
- added R117: 1k, Resistor_THT:R_Axial_DIN0207_L6.3mm_D2.5mm_P10.16mm_Horizontal, F.Cu at (177.5, 57.4)
- added R118: 1k, Resistor_THT:R_Axial_DIN0207_L6.3mm_D2.5mm_P10.16mm_Horizontal, F.Cu at (182.5, 67.6)
- added R201: 1k, Resistor_THT:R_Axial_DIN0207_L6.3mm_D2.5mm_P10.16mm_Horizontal, F.Cu at (138.6, 122.5)
- added R202: 1k, Resistor_THT:R_Axial_DIN0207_L6.3mm_D2.5mm_P10.16mm_Horizontal, F.Cu at (128.4, 126.0)
- added R203: 1k, Resistor_THT:R_Axial_DIN0207_L6.3mm_D2.5mm_P10.16mm_Horizontal, F.Cu at (138.6, 119.0)
- added R204: 1k, Resistor_THT:R_Axial_DIN0207_L6.3mm_D2.5mm_P10.16mm_Horizontal, F.Cu at (128.4, 115.5)
- added R205: 1k, Resistor_THT:R_Axial_DIN0207_L6.3mm_D2.5mm_P10.16mm_Horizontal, F.Cu at (138.6, 106.5)
- added R206: 1k, Resistor_THT:R_Axial_DIN0207_L6.3mm_D2.5mm_P10.16mm_Horizontal, F.Cu at (179.8, 91.5)
- added R207: 1k, Resistor_THT:R_Axial_DIN0207_L6.3mm_D2.5mm_P10.16mm_Horizontal, F.Cu at (175.8, 101.6)
- added R208: 1k, Resistor_THT:R_Axial_DIN0207_L6.3mm_D2.5mm_P10.16mm_Horizontal, F.Cu at (183.8, 91.4)
- added R209: 1k, Resistor_THT:R_Axial_DIN0207_L6.3mm_D2.5mm_P10.16mm_Horizontal, F.Cu at (188.0, 101.6)
- added R210: 1k, Resistor_THT:R_Axial_DIN0207_L6.3mm_D2.5mm_P10.16mm_Horizontal, F.Cu at (161.9, 113.7)
- added U101: ESP32-WROOM-32, Mainboard:diymore-ESP32-WROOM-32-Devboard, F.Cu at (139.6, 52.0)
- added U201: DRV8834, Mainboard:Polulu_DRV8834, F.Cu at (122.3, 125.4)
- added U202: DRV8834, Mainboard:Polulu_DRV8834, F.Cu at (179.0, 108.5)
Routing:
- net VDD: track 0.00 -> 220.5 mm
- net VBUS: track 0.00 -> 170.1 mm
- net /~{FAULT_RIGHT}: track 0.00 -> 87.1 mm
- net Net-(U101-D13): track 0.00 -> 80.6 mm
- net Net-(U101-D12): track 0.00 -> 72.5 mm
- net /DIR_RIGHT: track 0.00 -> 70.0 mm
- net /STEP_RIGHT: track 0.00 -> 67.2 mm
- net Net-(U101-D14): track 0.00 -> 63.7 mm
- net Net-(U101-D15): track 0.00 -> 57.8 mm
- net Net-(U101-D2): track 0.00 -> 50.3 mm
- net Net-(U101-D4): track 0.00 -> 42.8 mm
- net /SCL: track 0.00 -> 32.9 mm
- net /SDA: track 0.00 -> 29.0 mm
- net /~{FAULT_LEFT}: track 0.00 -> 25.2 mm
- net Net-(U202-M1): track 0.00 -> 18.9 mm
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- added copper zone on B.Cu, net GND
- added copper zone on F.Cu, net GND
Other:
- board outline added: 100 x 81 mm
