File: example/charging_station/Mainboard_V1/Mainboard_V1.kicad_pcb (KiCad board)
At the start: 2 copper layers, 100 x 81 mm, 33 parts, among them J104 Conn_01x04_Pin, J107 Conn_01x08_Pin, U101 ESP32-WROOM-32, U201 DRV8834, U202 DRV8834

Commit message: PCB V1 first manufactured prototype
Connections:
- C201 pad 2: (no net) -> GND
- C202 pad 2: (no net) -> GND
- U201 pad 10: (no net) -> GND
- U202 pad 10: (no net) -> GND
Other:
- board text added: "Mose Schmiedel"

Commit message: PCB updates
Connections:
- C101 pad 2: (no net) -> GND
Changed lines of the file:
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@@
 		(tenting front back)
 		(pcbplotparams
-			(layerselection 0x00000000_00000000_55555555_5755f5ff)
+			(layerselection 0x00000000_00000000_55555555_57555555)
 			(plot_on_all_layers_selection 0x00000000_00000000_00000000_00000000)
 			(disableapertmacros no)
@@
 			(outputformat 1)
 			(mirror no)
-			(drillshape 1)
+			(drillshape 0)
 			(scaleselection 1)
-			(outputdirectory "")
+			(outputdirectory "gerber/")
 		)
 	)
@@
 			(layers "*.Cu" "*.Mask")
 			(remove_unused_layers no)
+			(net 1 "GND")
 			(pintype "passive")
 		)
